Commit message: Adds lidar and ground truth odometry for ros_gz

File: leo_description/urdf/macros.xacro (robot description, xacro)
@@ -155,4 +155,5 @@
     </xacro:if>
     <link name="${link_prefix}camera_frame"/>
+    <link name="${link_prefix}lidar_frame"/>
     <link name="${link_prefix}camera_optical_frame"/>
     <link name="${link_prefix}imu_frame"/>
@@ -247,4 +248,9 @@
       </joint>
     </xacro:if>
+    <joint name="${joint_prefix}lidar_joint" type="fixed">
+      <origin xyz="0.0971 0 -0.0427" rpy="0 0.2094 0"/>
+      <parent link="${link_prefix}base_link"/>
+      <child link="${link_prefix}lidar_frame"/>
+    </joint>
     <joint name="${joint_prefix}camera_joint" type="fixed">
       <origin xyz="0.0971 0 -0.0427" rpy="0 0.2094 0"/>
@@ -453,5 +459,37 @@
           <visualize>true</visualize>
           <topic>${link_prefix}camera/image_raw</topic>
-          <ignition_frame_id>${link_prefix}camera_frame</ignition_frame_id>
+          <gz_frame_id>${link_prefix}camera_frame</gz_frame_id>
+      </sensor>
+    </gazebo>
+    <!-- fake lidar for sim-->
+    <gazebo reference="${link_prefix}lidar_frame">
+      <sensor name='lidar_frame' type='gpu_lidar'>
+        <pose relative_to='lidar_frame'>0 0 0 0 0 0</pose>
+        <topic>${link_prefix}scan</topic>
+        <update_rate>10</update_rate>
+        <ray>
+          <scan>
+            <horizontal>
+              <samples>640</samples>
+              <resolution>1</resolution>
+              <min_angle>-1.396263</min_angle>
+              <max_angle>1.396263</max_angle>
+            </horizontal>
+            <vertical>
+              <samples>1</samples>
+              <resolution>0.01</resolution>
+              <min_angle>1</min_angle>
+              <max_angle>1</max_angle>
+            </vertical>
+          </scan>
+          <range>
+            <min>0.08</min>
+            <max>10.0</max>
+            <resolution>0.01</resolution>
+          </range>
+        </ray>
+        <always_on>true</always_on>
+        <visualize>true</visualize>
+        <gz_frame_id>${link_prefix}lidar_frame</gz_frame_id>
       </sensor>
     </gazebo>
@@ -477,5 +515,5 @@
         <topic>${link_prefix}imu/data_raw</topic>
         <always_on>1</always_on>
-        <ignition_frame_id>${link_prefix}imu_frame</ignition_frame_id>
+        <gz_frame_id>${link_prefix}imu_frame</gz_frame_id>
       </sensor>
     </gazebo>
@@ -494,10 +532,15 @@
         <odom_publish_frequency>20</odom_publish_frequency>
         <topic>${link_prefix}cmd_vel</topic>
-        <odom_topic>${link_prefix}odom</odom_topic>
-        <tf_topic>${link_prefix}tf</tf_topic>
         <max_linear_acceleration>2.5</max_linear_acceleration>
         <max_angular_acceleration>3</max_angular_acceleration>
         <min_linear_acceleration>-2.5</min_linear_acceleration>
         <min_angular_acceleration>-3</min_angular_acceleration>
+      </plugin>
+      <plugin filename="libignition-gazebo-odometry-publisher-system.so" name="ignition::gazebo::systems::OdometryPublisher">
+        <update_frequency>10</update_frequency>
+        <odom_topic>${link_prefix}true_pose</odom_topic>
+        <odom_frame>world</odom_frame>
+        <robot_base_frame>${link_prefix}base_footprint</robot_base_frame>
+        <tf_topic>${link_prefix}tf</tf_topic>
       </plugin>
     </gazebo>

Commit message: Fix robot_ns tag

File: leo_description/urdf/macros.xacro (robot description, xacro)
@@ -98,4 +98,5 @@
     </xacro:if>
     <link name="${link_prefix}base_link">
+      <pose>0 0 0.19783 0 0 0</pose>
       <inertial>
         <mass value="1.584994"/>
@@ -158,4 +159,44 @@
     <link name="${link_prefix}camera_optical_frame"/>
     <link name="${link_prefix}imu_frame"/>
+    <link name="${joint_prefix}rotor_FL_link">
+      <inertial>
+        <mass value="0.1"/>
+        <origin xyz="0 0 0"/>
+        <inertia
+          ixx="0.0001" ixy="0" ixz="0"
+          iyy="0.0001" iyz="0"
+          izz="0.0001"/>
+      </inertial>
+    </link>
+    <link name="${joint_prefix}rotor_FR_link">
+      <inertial>
+        <mass value="0.1"/>
+        <origin xyz="0 0 0"/>
+        <inertia
+          ixx="0.0001" ixy="0" ixz="0"
+          iyy="0.0001" iyz="0"
+          izz="0.0001"/>
+      </inertial>
+    </link>
+    <link name="${joint_prefix}rotor_RL_link">
+      <inertial>
+        <mass value="0.1"/>
+        <origin xyz="0 0 0"/>
+        <inertia
+          ixx="0.0001" ixy="0" ixz="0"
+          iyy="0.0001" iyz="0"
+          izz="0.0001"/>
+      </inertial>
+    </link>
+    <link name="${joint_prefix}rotor_RR_link">
+      <inertial>
+        <mass value="0.1"/>
+        <origin xyz="0 0 0"/>
+        <inertia
+          ixx="0.0001" ixy="0" ixz="0"
+          iyy="0.0001" iyz="0"
+          izz="0.0001"/>
+      </inertial>
+    </link>
     <!-- JOINTS -->
     <xacro:if value="${footprint_link}">
@@ -187,5 +228,5 @@
       <limit effort="100.0" lower="-0.24" upper="0.24" velocity="100.0"/>
       <dynamics friction="1.0" damping="0.1"/>
-      <mimic joint="rocker_L_joint"/>
+      <mimic joint="${joint_prefix}rocker_L_joint"/>
     </joint>
     <joint name="${joint_prefix}wheel_FL_joint" type="continuous">
@@ -265,15 +306,37 @@
     <joint name="${joint_prefix}imu_joint" type="fixed">
       <origin xyz="${imu_translation}" rpy="0 0 0"/>
-      <parent link="${link_prefix}base_link"/>
+      <parent link="${link_prefix}base_footprint"/>
       <child link="${link_prefix}imu_frame"/>
+    </joint>
+    <joint name="${joint_prefix}rotor_FL_joint" type="continuous">
+      <parent link="${link_prefix}base_link"/>
+      <child link="${link_prefix}rotor_FL_link"/>
+      <origin xyz="0.2 0.2 0.1" rpy="0 0 0"/>
+      <axis xyz="0 0 1"/>
+    </joint>
+    <joint name="${joint_prefix}rotor_FR_joint" type="continuous">
+      <parent link="${link_prefix}base_link"/>
+      <child link="${link_prefix}rotor_FR_link"/>
+      <origin xyz="0.2 -0.2 0.1" rpy="0 0 0"/>
+      <axis xyz="0 0 1"/>
+    </joint>
+    <joint name="${joint_prefix}rotor_RL_joint" type="continuous">
+      <parent link="${link_prefix}base_link"/>
+      <child link="${link_prefix}rotor_RL_link"/>
+      <origin xyz="-0.2 0.2 0.1" rpy="0 0 0"/>
+      <axis xyz="0 0 1"/>
+    </joint>
+    <joint name="${joint_prefix}rotor_RR_joint" type="continuous">
+      <parent link="${link_prefix}base_link"/>
+      <child link="${link_prefix}rotor_RR_link"/>
+      <origin xyz="-0.2 -0.2 0.1" rpy="0 0 0"/>
+      <axis xyz="0 0 1"/>
     </joint>
   </xacro:macro>
   <!-- LEO GAZEBO -->
   <xacro:macro name="leo_gazebo"
-               params="robot_ns:='''">
-    <xacro:property name="link_prefix" value=""/>
-    <xacro:if value="${robot_ns != '' and robot_ns != '/'}">
-      <xacro:property name="link_prefix" value="${robot_ns}/"/>
-    </xacro:if>
+               params="robot_ns:=''
+               link_prefix:=''
+               joint_prefix:=''">
     <!-- base ODE properties -->
     <gazebo reference="${link_prefix}base_footprint">
@@ -497,6 +560,6 @@
     <gazebo>
       <plugin name="leo_gz::DifferentialSystem" filename="libleo_gz_differential_plugin.so">
-        <jointA>rocker_L_joint</jointA>
-        <jointB>rocker_R_joint</jointB>
+        <jointA>${joint_prefix}rocker_L_joint</jointA>
+        <jointB>${joint_prefix}rocker_R_joint</jointB>
         <forceConstant>100.0</forceConstant>
       </plugin>
@@ -522,8 +585,8 @@
         filename="libignition-gazebo-diff-drive-system.so"
         name="ignition::gazebo::systems::DiffDrive">
-        <left_joint>wheel_FL_joint</left_joint>
-        <right_joint>wheel_FR_joint</right_joint>
-        <left_joint>wheel_RL_joint</left_joint>
-        <right_joint>wheel_RR_joint</right_joint>
+        <left_joint>${joint_prefix}wheel_FL_joint</left_joint>
+        <right_joint>${joint_prefix}wheel_FR_joint</right_joint>
+        <left_joint>${joint_prefix}wheel_RL_joint</left_joint>
+        <right_joint>${joint_prefix}wheel_RR_joint</right_joint>
         <wheel_separation>0.358</wheel_separation>
         <wheel_radius>0.0625</wheel_radius>
@@ -531,5 +594,5 @@
         <child_frame_id>${link_prefix}base_footprint</child_frame_id>
         <odom_publish_frequency>20</odom_publish_frequency>
-        <topic>${link_prefix}cmd_vel</topic>
+        <topic>${robot_ns}/cmd_vel</topic>
         <max_linear_acceleration>2.5</max_linear_acceleration>
         <max_angular_acceleration>3</max_angular_acceleration>
@@ -545,4 +608,44 @@
       </plugin>
     </gazebo>
+    <gazebo>
+      <plugin
+        filename="ignition-gazebo-multicopter-control-system"
+        name="ignition::gazebo::systems::MulticopterVelocityControl">
+        <robotNamespace>${robot_ns}</robotNamespace>
+        <commandSubTopic>cmd_vel</commandSubTopic>
+        <enableSubTopic>drone_enable</enableSubTopic>
+        <comLinkName>${link_prefix}base_link</comLinkName>
+        <velocityGain>4.0 4.0 4.0</velocityGain>
+        <attitudeGain>4 5 0.3</attitudeGain>
+        <angularRateGain>0.6 0.8 0.3</angularRateGain>
+        <maximumLinearAcceleration>5 5 5</maximumLinearAcceleration>
+        <rotorConfiguration>
+          <rotor>
+              <jointName>${joint_prefix}rotor_FL_joint</jointName>
+              <forceConstant>1.5e-05</forceConstant>
+              <momentConstant>0.016</momentConstant>
+              <direction>1</direction>
+          </rotor>
+          <rotor>
+              <jointName>${joint_prefix}rotor_FR_joint</jointName>
+              <forceConstant>1.5e-05</forceConstant>
+              <momentConstant>0.016</momentConstant>
+              <direction>-1</direction>
+          </rotor>
+          <rotor>
+              <jointName>${joint_prefix}rotor_RL_joint</jointName>
+              <forceConstant>1.5e-05</forceConstant>
+              <momentConstant>0.016</momentConstant>
+              <direction>-1</direction>
+          </rotor>
+          <rotor>
+              <jointName>${joint_prefix}rotor_RR_joint</jointName>
+              <forceConstant>1.5e-05</forceConstant>
+              <momentConstant>0.016</momentConstant>
+              <direction>1</direction>
+          </rotor>
+        </rotorConfiguration>
+      </plugin>
+    </gazebo>
   </xacro:macro>
   <xacro:macro name="leo_sim"
@@ -552,12 +655,18 @@
                        mecanum_wheels:=false">
     <xacro:property name="link_prefix" value=""/>
+    <xacro:property name="joint_prefix" value=""/>
     <xacro:if value="${robot_ns != '' and robot_ns != '/'}">
       <xacro:property name="link_prefix" value="${robot_ns}/"/>
+      <xacro:property name="joint_prefix" value="${robot_ns}/"/>
     </xacro:if>
     <xacro:leo default_antenna="${default_antenna}"
                rockers_fixed="false"
                link_prefix="${link_prefix}"
+               joint_prefix="${joint_prefix}"
                mecanum_wheels="${mecanum_wheels}"/>
-    <xacro:leo_gazebo robot_ns="${robot_ns}"/>
+    <xacro:leo_gazebo robot_ns="${robot_ns}"
+                      link_prefix="${link_prefix}"
+                      joint_prefix="${joint_prefix}"
+              />
     <xacro:if value="${fixed}">
       <link name="world"/>
