Commit message: Updated description

File: leo_description/urdf/macros.xacro (robot description, xacro)
@@ -4,11 +4,8 @@
                params="default_antenna:=true
                        rockers_fixed:=true
-                       footprint_link:=true
-                       link_prefix:=''
-                       joint_prefix:=''
                        imu_translation:='0.0628 -0.0314 -0.0393'
                        mecanum_wheels:=false">
     <xacro:macro name="rocker_link" params="name">
-      <link name="${link_prefix}rocker_${name}_link">
+      <link name="rocker_${name}_link">
         <inertial>
           <mass value="1.387336"/>
@@ -21,10 +18,10 @@
         <visual>
           <geometry>
-            <mesh filename="package://leo_description/models/Rocker.dae"/>
+            <mesh filename="package://Rocker.dae"/>
           </geometry>
         </visual>
         <collision>
           <geometry>
-            <mesh filename="package://leo_description/models/Rocker_outline.stl"/>
+            <mesh filename="package://Rocker_outline.stl"/>
           </geometry>
         </collision>
@@ -32,5 +29,5 @@
     </xacro:macro>
     <xacro:macro name="wheel_link" params="name model">
-      <link name="${link_prefix}wheel_${name}_link">
+      <link name="wheel_${name}_link">
         <inertial>
           <mass value="0.283642"/>
@@ -43,5 +40,5 @@
         <visual>
           <geometry>
-            <mesh filename="package://leo_description/models/Wheel${model}.dae"/>
+            <mesh filename="package://Wheel${model}.dae"/>
           </geometry>
         </visual>
@@ -60,5 +57,5 @@
         <collision>
           <geometry>
-            <mesh filename="package://leo_description/models/Wheel_outline.stl"/>
+            <mesh filename="package://Wheel_outline.stl"/>
           </geometry>
         </collision>
@@ -66,5 +63,5 @@
     </xacro:macro>
     <xacro:macro name="mecanum_wheel_link" params="name model">
-      <link name="${link_prefix}wheel_${name}_link">
+      <link name="wheel_${name}_link">
         <inertial>
           <mass value="0.672214"/>
@@ -77,5 +74,5 @@
         <visual>
           <geometry>
-            <mesh filename="package://leo_description/models/WheelMecanum${model}.dae"/>
+            <mesh filename="package://WheelMecanum${model}.dae"/>
           </geometry>
         </visual>
@@ -88,5 +85,5 @@
         <collision>
           <geometry>
-            <mesh filename="package://leo_description/models/Mecanum_wheel_outline.stl"/>
+            <mesh filename="package://Mecanum_wheel_outline.stl"/>
           </geometry>
         </collision>
@@ -94,8 +91,5 @@
     </xacro:macro>
     <!-- LINKS -->
-    <xacro:if value="${footprint_link}">
-      <link name="${link_prefix}base_footprint"/>
-    </xacro:if>
-    <link name="${link_prefix}base_link">
+    <link name="base_link">
       <pose>0 0 0.19783 0 0 0</pose>
       <inertial>
@@ -109,10 +103,10 @@
       <visual>
         <geometry>
-          <mesh filename="package://leo_description/models/Chassis.dae"/>
+          <mesh filename="package://Chassis.dae"/>
         </geometry>
       </visual>
       <collision>
         <geometry>
-          <mesh filename="package://leo_description/models/Chassis_outline.stl"/>
+          <mesh filename="package://Chassis_outline.stl"/>
         </geometry>
       </collision>
@@ -133,5 +127,5 @@
     </xacro:unless>
     <xacro:if value="${default_antenna}">
-      <link name="${link_prefix}antenna_link">
+      <link name="antenna_link">
         <inertial>
           <mass value="0.001237"/>
@@ -144,5 +138,5 @@
         <visual>
           <geometry>
-            <mesh filename="package://leo_description/models/Antenna.dae"/>
+            <mesh filename="package://Antenna.dae"/>
           </geometry>
         </visual>
@@ -155,56 +149,9 @@
       </link>
     </xacro:if>
-    <link name="${link_prefix}camera_frame"/>
-    <link name="${link_prefix}lidar_frame"/>
-    <link name="${link_prefix}camera_optical_frame"/>
-    <link name="${link_prefix}imu_frame"/>
-    <link name="${joint_prefix}rotor_FL_link">
-      <inertial>
-        <mass value="0.1"/>
-        <origin xyz="0 0 0"/>
-        <inertia
-          ixx="0.0001" ixy="0" ixz="0"
-          iyy="0.0001" iyz="0"
-          izz="0.0001"/>
-      </inertial>
-    </link>
-    <link name="${joint_prefix}rotor_FR_link">
-      <inertial>
-        <mass value="0.1"/>
-        <origin xyz="0 0 0"/>
-        <inertia
-          ixx="0.0001" ixy="0" ixz="0"
-          iyy="0.0001" iyz="0"
-          izz="0.0001"/>
-      </inertial>
-    </link>
-    <link name="${joint_prefix}rotor_RL_link">
-      <inertial>
-        <mass value="0.1"/>
-        <origin xyz="0 0 0"/>
-        <inertia
-          ixx="0.0001" ixy="0" ixz="0"
-          iyy="0.0001" iyz="0"
-          izz="0.0001"/>
-      </inertial>
-    </link>
-    <link name="${joint_prefix}rotor_RR_link">
-      <inertial>
-        <mass value="0.1"/>
-        <origin xyz="0 0 0"/>
-        <inertia
-          ixx="0.0001" ixy="0" ixz="0"
-          iyy="0.0001" iyz="0"
-          izz="0.0001"/>
-      </inertial>
-    </link>
+    <link name="camera_frame"/>
+    <link name="lidar_frame"/>
+    <link name="camera_optical_frame"/>
+    <link name="imu_frame"/>
     <!-- JOINTS -->
-    <xacro:if value="${footprint_link}">
-      <joint name="${joint_prefix}base_joint" type="fixed">
-        <origin xyz="0 0 0.19783" rpy="0 0 0"/>
-        <parent link="${link_prefix}base_footprint"/>
-        <child link="${link_prefix}base_link"/>
-      </joint>
-    </xacro:if>
     <xacro:if value="${rockers_fixed}">
       <xacro:property name="rockers_joint_type" value="fixed"/>
@@ -213,22 +160,22 @@
       <xacro:property name="rockers_joint_type" value="revolute"/>
     </xacro:unless>
-    <joint name="${joint_prefix}rocker_L_joint" type="${rockers_joint_type}">
+    <joint name="rocker_L_joint" type="${rockers_joint_type}">
       <origin xyz="0.00263 0.14167 -0.04731" rpy="0 0 ${pi}"/>
-      <parent link="${link_prefix}base_link"/>
-      <child link="${link_prefix}rocker_L_link"/>
+      <parent link="base_link"/>
+      <child link="rocker_L_link"/>
       <axis xyz="0 1 0"/>
       <limit effort="100.0" lower="-0.24" upper="0.24" velocity="100.0"/>
       <dynamics friction="1.0" damping="0.1"/>
     </joint>
-    <joint name="${joint_prefix}rocker_R_joint" type="${rockers_joint_type}">
+    <joint name="rocker_R_joint" type="${rockers_joint_type}">
       <origin xyz="0.00263 -0.14167 -0.04731" rpy="0 0 0"/>
-      <parent link="${link_prefix}base_link"/>
-      <child link="${link_prefix}rocker_R_link"/>
+      <parent link="base_link"/>
+      <child link="rocker_R_link"/>
       <axis xyz="0 1 0"/>
       <limit effort="100.0" lower="-0.24" upper="0.24" velocity="100.0"/>
       <dynamics friction="1.0" damping="0.1"/>
-      <mimic joint="${joint_prefix}rocker_L_joint"/>
-    </joint>
-    <joint name="${joint_prefix}wheel_FL_joint" type="continuous">
+      <mimic joint="rocker_L_joint"/>
+    </joint>
+    <joint name="wheel_FL_joint" type="continuous">
       <xacro:if value="${mecanum_wheels}">
         <origin xyz="-0.15256 -0.00884 -0.08802" rpy="0 0 0"/>
@@ -237,11 +184,11 @@
         <origin xyz="-0.15256 -0.08214 -0.08802" rpy="0 0 0"/>
       </xacro:unless>
-      <parent link="${link_prefix}rocker_L_link"/>
-      <child link="${link_prefix}wheel_FL_link"/>
+      <parent link="rocker_L_link"/>
+      <child link="wheel_FL_link"/>
       <axis xyz="0 -1 0"/>
       <limit effort="2.0" velocity="6.0"/>
       <dynamics friction="0.3125" damping="0.1"/>
     </joint>
-    <joint name="${joint_prefix}wheel_RL_joint" type="continuous">
+    <joint name="wheel_RL_joint" type="continuous">
       <xacro:if value="${mecanum_wheels}">
         <origin xyz="0.15256 -0.00884 -0.08802" rpy="0 0 0"/>
@@ -250,11 +197,11 @@
         <origin xyz="0.15256 -0.08214 -0.08802" rpy="0 0 0"/>
       </xacro:unless>
-      <parent link="${link_prefix}rocker_L_link"/>
-      <child link="${link_prefix}wheel_RL_link"/>
+      <parent link="rocker_L_link"/>
+      <child link="wheel_RL_link"/>
       <axis xyz="0 -1 0"/>
       <limit effort="2.0" velocity="6.0"/>
       <dynamics friction="0.3125" damping="0.1"/>
     </joint>
-    <joint name="${joint_prefix}wheel_FR_joint" type="continuous">
+    <joint name="wheel_FR_joint" type="continuous">
       <xacro:if value="${mecanum_wheels}">
         <origin xyz="0.15256 -0.00884 -0.08802" rpy="0 0 0"/>
@@ -263,11 +210,11 @@
         <origin xyz="0.15256 -0.08214 -0.08802" rpy="0 0 0"/>
       </xacro:unless>
-      <parent link="${link_prefix}rocker_R_link"/>
-      <child link="${link_prefix}wheel_FR_link"/>
+      <parent link="rocker_R_link"/>
+      <child link="wheel_FR_link"/>
       <axis xyz="0 1 0"/>
       <limit effort="2.0" velocity="6.0"/>
       <dynamics friction="0.3125" damping="0.1"/>
     </joint>
-    <joint name="${joint_prefix}wheel_RR_joint" type="continuous">
+    <joint name="wheel_RR_joint" type="continuous">
       <xacro:if value="${mecanum_wheels}">
         <origin xyz="-0.15256 -0.00884 -0.08802" rpy="0 0 0"/>
@@ -276,6 +223,6 @@
         <origin xyz="-0.15256 -0.08214 -0.08802" rpy="0 0 0"/>
       </xacro:unless>
-      <parent link="${link_prefix}rocker_R_link"/>
-      <child link="${link_prefix}wheel_RR_link"/>
+      <parent link="rocker_R_link"/>
+      <child link="wheel_RR_link"/>
       <axis xyz="0 1 0"/>
       <limit effort="2.0" velocity="6.0"/>
@@ -283,62 +230,36 @@
     </joint>
     <xacro:if value="${default_antenna}">
-      <joint name="${joint_prefix}antenna_joint" type="fixed">
+      <joint name="antenna_joint" type="fixed">
         <origin xyz="-0.0052 0.056 -0.0065" rpy="0 0 0"/>
-        <parent link="${link_prefix}base_link"/>
-        <child link="${link_prefix}antenna_link"/>
+        <parent link="base_link"/>
+        <child link="antenna_link"/>
       </joint>
     </xacro:if>
-    <joint name="${joint_prefix}lidar_joint" type="fixed">
+    <joint name="lidar_joint" type="fixed">
+      <origin xyz="0.0971 0 -0.0427" rpy="0 0.7 0"/>
+      <parent link="base_link"/>
+      <child link="lidar_frame"/>
+    </joint>
+    <joint name="camera_joint" type="fixed">
       <origin xyz="0.0971 0 -0.0427" rpy="0 0.2094 0"/>
-      <parent link="${link_prefix}base_link"/>
-      <child link="${link_prefix}lidar_frame"/>
-    </joint>
-    <joint name="${joint_prefix}camera_joint" type="fixed">
-      <origin xyz="0.0971 0 -0.0427" rpy="0 0.2094 0"/>
-      <parent link="${link_prefix}base_link"/>
-      <child link="${link_prefix}camera_frame"/>
-    </joint>
-    <joint name="${joint_prefix}camera_optical_joint" type="fixed">
+      <parent link="base_link"/>
+      <child link="camera_frame"/>
+    </joint>
+    <joint name="camera_optical_joint" type="fixed">
       <origin xyz="0 0 0" rpy="-${pi/2} 0.0 -${pi/2}"/>
-      <parent link="${link_prefix}camera_frame"/>
-      <child link="${link_prefix}camera_optical_frame"/>
-    </joint>
-    <joint name="${joint_prefix}imu_joint" type="fixed">
+      <parent link="camera_frame"/>
+      <child link="camera_optical_frame"/>
+    </joint>
+    <joint name="imu_joint" type="fixed">
       <origin xyz="${imu_translation}" rpy="0 0 0"/>
-      <parent link="${link_prefix}base_footprint"/>
-      <child link="${link_prefix}imu_frame"/>
-    </joint>
-    <joint name="${joint_prefix}rotor_FL_joint" type="continuous">
-      <parent link="${link_prefix}base_link"/>
-      <child link="${link_prefix}rotor_FL_link"/>
-      <origin xyz="0.2 0.2 0.1" rpy="0 0 0"/>
-      <axis xyz="0 0 1"/>
-    </joint>
-    <joint name="${joint_prefix}rotor_FR_joint" type="continuous">
-      <parent link="${link_prefix}base_link"/>
-      <child link="${link_prefix}rotor_FR_link"/>
-      <origin xyz="0.2 -0.2 0.1" rpy="0 0 0"/>
-      <axis xyz="0 0 1"/>
-    </joint>
-    <joint name="${joint_prefix}rotor_RL_joint" type="continuous">
-      <parent link="${link_prefix}base_link"/>
-      <child link="${link_prefix}rotor_RL_link"/>
-      <origin xyz="-0.2 0.2 0.1" rpy="0 0 0"/>
-      <axis xyz="0 0 1"/>
-    </joint>
-    <joint name="${joint_prefix}rotor_RR_joint" type="continuous">
-      <parent link="${link_prefix}base_link"/>
-      <child link="${link_prefix}rotor_RR_link"/>
-      <origin xyz="-0.2 -0.2 0.1" rpy="0 0 0"/>
-      <axis xyz="0 0 1"/>
+      <parent link="base_link"/>
+      <child link="imu_frame"/>
     </joint>
   </xacro:macro>
   <!-- LEO GAZEBO -->
   <xacro:macro name="leo_gazebo"
-               params="robot_ns:=''
-               link_prefix:=''
-               joint_prefix:=''">
+               params="robot_ns:=''">
     <!-- base ODE properties -->
-    <gazebo reference="${link_prefix}base_footprint">
+    <gazebo reference="base_link">
       <collision>
         <surface>
@@ -357,5 +278,5 @@
       </collision>
     </gazebo>
-    <gazebo reference="${link_prefix}base_link">
+    <gazebo reference="base_link">
       <collision>
         <surface>
@@ -375,5 +296,5 @@
     </gazebo>
     <!-- rocker ODE properties -->
-    <gazebo reference="${link_prefix}rocker_L_link">
+    <gazebo reference="rocker_L_link">
       <collision>
         <surface>
@@ -392,5 +313,5 @@
       </collision>
     </gazebo>
-    <gazebo reference="${link_prefix}rocker_R_link">
+    <gazebo reference="rocker_R_link">
       <collision>
         <surface>
@@ -410,5 +331,5 @@
     </gazebo>
     <!-- wheel ODE properties -->
-    <gazebo reference="${link_prefix}wheel_FL_link">
+    <gazebo reference="wheel_FL_link">
       <collision>
         <surface>
@@ -417,18 +338,17 @@
               <mu>1</mu>
               <mu2>1</mu2>
-              <slip1>0.035</slip1>
-              <slip2>0</slip2>
-              <fdir1>0 0 1</fdir1>
+              <slip1>0.01</slip1>
+              <slip2>0.01</slip2>
             </ode>
             <bullet>
               <friction>1</friction>
               <friction2>1</friction2>
-              <rolling_friction>0.1</rolling_friction>
-            </bullet>
-          </friction>
-        </surface>
-      </collision>
-    </gazebo>
-    <gazebo reference="${link_prefix}wheel_FR_link">
+              <rolling_friction>0</rolling_friction>
+            </bullet>
+          </friction>
+        </surface>
+      </collision>
+    </gazebo>
+    <gazebo reference="wheel_FR_link">
       <collision>
         <surface>
@@ -437,18 +357,17 @@
               <mu>1</mu>
               <mu2>1</mu2>
-              <slip1>0.035</slip1>
-              <slip2>0</slip2>
-              <fdir1>0 0 1</fdir1>
+              <slip1>0.01</slip1>
+              <slip2>0.01</slip2>
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